Commit message: Changed asset placement in scene

File: assets/demo/robot.urdf (robot description, URDF)
Before this commit: robot Robot, 1 links, 0 joints
Links:
- added link back_caster_wheel, mass 2; collision sphere radius=0.02; visual sphere radius=0.02
- added link left_wheel, mass 1; collision cylinder length=0.02 radius=0.05; visual box size=0.02 0.07 0.02
- added link right_wheel, mass 1; collision cylinder length=0.02 radius=0.05; visual box size=0.02 0.07 0.02
- link base_link: mass None -> 1; geometry collision cylinder length=0.1 radius=0.12; visual box size=0.05 0.1 0.01
Joints:
- added joint back_caster_joint: type fixed, parent base_link, child back_caster_wheel, origin xyz=-0.10 0.0 0.020 rpy=0 0 0
- added joint left_joint: type continuous, parent base_link, child left_wheel, origin xyz=0.05 0.13 0.05 rpy=0 0 0, axis 0.0 1.0 0.0, limit effort=10 velocity=5.0
- added joint right_joint: type continuous, parent base_link, child right_wheel, origin xyz=0.05 -0.12 0.05 rpy=0 0 0, axis 0.0 1.0 0.0, limit effort=10 velocity=5.0
