Commit message: Added Mecanum wheel feature

File: assets/demo/robot_mecanum.urdf (robot description, URDF)
Before this commit: robot Robot mecanum wheels, 5 links, 4 joints
Links:
- link back_left_wheel: mass None -> 0.1
- link back_right_wheel: mass None -> 0.1
- link front_left_wheel: mass None -> 0.1
- link front_right_wheel: mass None -> 0.1
Joints:
- joint back_left_joint: limit effort=10 velocity=5.0 -> effort=100 velocity=5.0; origin xyz=-0.05 0.13 0.03 rpy=0 0 0 -> xyz=-0.11 0.11 0.03 rpy=0 0 0
- joint back_right_joint: limit effort=10 velocity=5.0 -> effort=100 velocity=5.0; origin xyz=-0.05 -0.13 0.03 rpy=0 0 0 -> xyz=-0.11 -0.11 0.03 rpy=0 0 0
- joint front_left_joint: limit effort=10 velocity=5.0 -> effort=100 velocity=5.0; origin xyz=0.05 0.13 0.03 rpy=0 0 0 -> xyz=0.11 0.11 0.03 rpy=0 0 0
- joint front_right_joint: limit effort=10 velocity=5.0 -> effort=100 velocity=5.0; origin xyz=0.05 -0.13 0.03 rpy=0 0 0 -> xyz=0.11 -0.11 0.03 rpy=0 0 0

Commit message: Changed Mecanum Wheel

File: assets/demo/robot_mecanum.urdf (robot description, URDF)
Before this commit: robot Robot Mecanum, 5 links, 4 joints
Links:
- link back_left_wheel: geometry visual cylinder length=0.1 radius=0.005
- link back_right_wheel: geometry visual cylinder length=0.1 radius=0.005
- link front_left_wheel: geometry visual cylinder length=0.1 radius=0.005
- link front_right_wheel: geometry visual cylinder length=0.1 radius=0.005
