Commit message: Fixed wrong scale for prismatic joint

File: assets/demo/robot_mecanum_wrench.urdf (robot description, URDF)
Before this commit: robot Robot Mecanum Wrench, 8 links, 7 joints
Joints:
- joint elevator_joint: limit lower=0.0 upper=0.1 effort=10000.0 velocity=5.0 -> lower=0.0 upper=0.1 effort=100 velocity=0.3

File: assets/demo/slider.urdf (robot description, URDF)
Before this commit: robot Slider, 2 links, 1 joints
Joints:
- joint arm servo: limit lower=-0.1 upper=0.2 velocity=1.0 -> lower=-0.1 upper=0.2 velocity=0.2

Commit message: Added Mecanum functions exposed to Python

File: assets/demo/robot_mecanum_wrench.urdf (robot description, URDF)
Before this commit: robot Robot Mecanum Wrench, 8 links, 7 joints
Links:
- link back_left_wheel: geometry visual cylinder length=0.1 radius=0.005
- link back_right_wheel: geometry visual cylinder length=0.1 radius=0.005
- link front_left_wheel: geometry visual cylinder length=0.1 radius=0.005
- link front_right_wheel: geometry visual cylinder length=0.1 radius=0.005

File: assets/demo/robot_wrench.urdf (robot description, URDF)
Before this commit: robot Robot with wrench, 8 links, 7 joints
Joints:
- joint elevator_joint: limit lower=0.0 upper=0.1 effort=10.0 velocity=5.0 -> lower=0.0 upper=0.1 effort=10.0 velocity=0.5
