Commit message: Changed differential robot

File: game/assets/demo/diff_robot.urdf (robot description, URDF)
Before this commit: robot Robot with 2 wheels, 4 links, 3 joints
Links:
- added link front_caster_wheel, mass 1; visual sphere radius=0.02
- link back_caster_wheel: mass 2 -> 1; geometry visual sphere radius=0.02
- link base_link: geometry visual box size=0.05 0.1 0.01; visual cylinder length=0.05 radius=0.18
- link left_wheel: geometry visual cylinder length=0.01 radius=0.03
- link right_wheel: geometry visual cylinder length=0.01 radius=0.03
Joints:
- added joint front_caster_joint: type pin, parent base_link, child front_caster_wheel, origin xyz=0.14 0.0 0.020 rpy=0 0 0
- joint back_caster_joint: origin xyz=-0.10 0.0 0.020 rpy=0 0 0 -> xyz=-0.14 0.0 0.021 rpy=0 0 0; type fixed -> pin
- joint left_joint: limit effort=10 velocity=5.0 -> effort=10 velocity=8.0; origin xyz=0.05 0.13 0.05 rpy=0 0 0 -> xyz=0.0 0.14 0.03 rpy=0 0 0
- joint right_joint: limit effort=10 velocity=5.0 -> effort=10 velocity=8.0; origin xyz=0.05 -0.12 0.05 rpy=0 0 0 -> xyz=0.0 -0.14 0.03 rpy=0 0 0
